Commit message: Revise URDF for jeep robot

File: urdf/mech/base.urdf.xacro (robot description, xacro)
@@ -8,5 +8,5 @@
         <geometry>
           <!-- box size="${length} ${width} ${height}"/ -->
-          <mesh filename="package://linorobot2_description/meshes/elsabot_jeep.stl" scale="1.0 1.0 1.0"/> -->
+          <mesh filename="package://elsabot_jeep/meshes/jeep_simple.stl" scale="1.0 1.0 1.0"/> -->
         </geometry>
         <material name="gray">

File: urdf/robots/2wd.urdf.xacro (robot description, xacro)
@@ -1,12 +1,12 @@
 <?xml version="1.0"?>
-<robot name="linorobot2_2wd" xmlns:xacro="http://ros.org/wiki/xacro">
-  <xacro:include filename="$(find linorobot2_description)/urdf/2wd_properties.urdf.xacro" />
-  <xacro:include filename="$(find linorobot2_description)/urdf/mech/base.urdf.xacro" />
-  <xacro:include filename="$(find linorobot2_description)/urdf/mech/wheel.urdf.xacro" />
-  <xacro:include filename="$(find linorobot2_description)/urdf/mech/caster_wheel.urdf.xacro" />
-  <xacro:include filename="$(find linorobot2_description)/urdf/sensors/imu.urdf.xacro" />
-  <xacro:include filename="$(find linorobot2_description)/urdf/sensors/generic_laser.urdf.xacro" />
-  <xacro:include filename="$(find linorobot2_description)/urdf/sensors/depth_sensor.urdf.xacro" />
-  <xacro:include filename="$(find linorobot2_description)/urdf/controllers/diff_drive.urdf.xacro" />
+<robot name="elsabot_jeep" xmlns:xacro="http://ros.org/wiki/xacro">
+  <xacro:include filename="$(find elsabot_jeep)/urdf/2wd_properties.urdf.xacro" />
+  <xacro:include filename="$(find elsabot_jeep)/urdf/mech/base.urdf.xacro" />
+  <xacro:include filename="$(find elsabot_jeep)/urdf/mech/wheel.urdf.xacro" />
+  <xacro:include filename="$(find elsabot_jeep)/urdf/mech/caster_wheel.urdf.xacro" />
+  <xacro:include filename="$(find elsabot_jeep)/urdf/sensors/imu.urdf.xacro" />
+  <xacro:include filename="$(find elsabot_jeep)/urdf/sensors/generic_laser.urdf.xacro" />
+  <xacro:include filename="$(find elsabot_jeep)/urdf/sensors/depth_sensor.urdf.xacro" />
+  <xacro:include filename="$(find elsabot_jeep)/urdf/controllers/diff_drive.urdf.xacro" />
   <xacro:base
     length="${base_length}"

File: urdf/robots/4wd.urdf.xacro (robot description, xacro)
@@ -1,12 +1,12 @@
 <?xml version="1.0"?>
-<robot name="linorobot2_2wd" xmlns:xacro="http://ros.org/wiki/xacro">
-  <xacro:include filename="$(find linorobot2_description)/urdf/4wd_properties.urdf.xacro" />
-  <xacro:include filename="$(find linorobot2_description)/urdf/mech/base.urdf.xacro" />
-  <xacro:include filename="$(find linorobot2_description)/urdf/mech/wheel.urdf.xacro" />
-  <xacro:include filename="$(find linorobot2_description)/urdf/sensors/imu.urdf.xacro" />
-  <xacro:include filename="$(find linorobot2_description)/urdf/sensors/generic_laser.urdf.xacro" />
-  <!--xacro:include filename="$(find linorobot2_description)/urdf/sensors/depth_sensor.urdf.xacro" /-->
-  <xacro:include filename="$(find linorobot2_description)/urdf/sensors/oakd_on_ptbase.urdf.xacro" />
-  <xacro:include filename="$(find linorobot2_description)/urdf/controllers/skid_steer.urdf.xacro" />
+<robot name="elsabot_jeep" xmlns:xacro="http://ros.org/wiki/xacro">
+  <xacro:include filename="$(find elsabot_jeep)/urdf/4wd_properties.urdf.xacro" />
+  <xacro:include filename="$(find elsabot_jeep)/urdf/mech/base.urdf.xacro" />
+  <xacro:include filename="$(find elsabot_jeep)/urdf/mech/wheel.urdf.xacro" />
+  <xacro:include filename="$(find elsabot_jeep)/urdf/sensors/imu.urdf.xacro" />
+  <xacro:include filename="$(find elsabot_jeep)/urdf/sensors/generic_laser.urdf.xacro" />
+  <!--xacro:include filename="$(find elsabot_jeep)/urdf/sensors/depth_sensor.urdf.xacro" /-->
+  <xacro:include filename="$(find elsabot_jeep)/urdf/sensors/oakd_on_ptbase.urdf.xacro" />
+  <xacro:include filename="$(find elsabot_jeep)/urdf/controllers/skid_steer.urdf.xacro" />
   <xacro:base
     length="${base_length}"

File: urdf/robots/jeep.urdf.xacro (robot description, xacro)
@@ -1,11 +1,12 @@
 <?xml version="1.0"?>
 <robot name="elsabot_jeep" xmlns:xacro="http://ros.org/wiki/xacro">
-  <xacro:include filename="$(find elsabot_jeep)/urdf/mecanum_properties.urdf.xacro" />
+  <xacro:include filename="$(find elsabot_jeep)/urdf/jeep_properties.urdf.xacro" />
   <xacro:include filename="$(find elsabot_jeep)/urdf/mech/base.urdf.xacro" />
-  <xacro:include filename="$(find elsabot_jeep)/urdf/mech/mecanum_wheel.urdf.xacro" />
+  <xacro:include filename="$(find elsabot_jeep)/urdf/mech/wheel.urdf.xacro" />
   <xacro:include filename="$(find elsabot_jeep)/urdf/sensors/imu.urdf.xacro" />
   <xacro:include filename="$(find elsabot_jeep)/urdf/sensors/generic_laser.urdf.xacro" />
-  <xacro:include filename="$(find elsabot_jeep)/urdf/sensors/depth_sensor.urdf.xacro" />
-  <xacro:include filename="$(find elsabot_jeep)/urdf/controllers/omni_drive.urdf.xacro" />
+  <!--xacro:include filename="$(find elsabot_jeep)/urdf/sensors/depth_sensor.urdf.xacro" /-->
+  <xacro:include filename="$(find elsabot_jeep)/urdf/sensors/oakd_on_ptbase.urdf.xacro" />
+  <!--xacro:include filename="$(find elsabot_jeep)/urdf/controllers/skid_steer.urdf.xacro" /-->
   <xacro:base
     length="${base_length}"
@@ -16,5 +17,5 @@
     wheel_pos_z="${wheel_pos_z}"
 />
-  <xacro:mecanum_wheel
+  <xacro:wheel
     side="front_left"
     radius="${wheel_radius}"
@@ -25,5 +26,5 @@
     mass="${wheel_mass}"
   />
-  <xacro:mecanum_wheel
+  <xacro:wheel
     side="front_right"
     radius="${wheel_radius}"
@@ -34,5 +35,5 @@
     mass="${wheel_mass}"
   />
-  <xacro:mecanum_wheel
+  <xacro:wheel
     side="rear_left"
     radius="${wheel_radius}"
@@ -43,5 +44,5 @@
     mass="${wheel_mass}"
   />
-  <xacro:mecanum_wheel
+  <xacro:wheel
     side="rear_right"
     radius="${wheel_radius}"
@@ -59,4 +60,8 @@
     <xacro:insert_block name="depth_sensor_pose" />
   </xacro:depth_sensor>
-  <xacro:omni_drive_controller/>
+  <!--xacro:diff_drive_controller
+    wheel_separation="${wheel_pos_y * 2}"
+    wheel_radius="${wheel_radius}"
+    wheel_torque="${wheel_torque}"
+  /-->
 </robot>

File: urdf/robots/square.urdf.xacro (robot description, xacro)
@@ -1,4 +1,4 @@
 <?xml version="1.0"?>
-<robot name="linorobot2_2wd" xmlns:xacro="http://ros.org/wiki/xacro">
+<robot name="elsabot_jeep" xmlns:xacro="http://ros.org/wiki/xacro">
   <xacro:property name="base_length" value="0.25" />
   <xacro:property name="base_width" value="0.25" />
@@ -14,11 +14,11 @@
   <xacro:property name="front_caster_wheel" value="false" />
   <xacro:property name="rear_caster_wheel" value="true" />
-  <xacro:include filename="$(find linorobot2_description)/urdf/mech/base.urdf.xacro" />
-  <xacro:include filename="$(find linorobot2_description)/urdf/mech/wheel.urdf.xacro" />
-  <xacro:include filename="$(find linorobot2_description)/urdf/mech/caster_wheel.urdf.xacro" />
-  <xacro:include filename="$(find linorobot2_description)/urdf/sensors/imu.urdf.xacro" />
-  <xacro:include filename="$(find linorobot2_description)/urdf/sensors/generic_laser.urdf.xacro" />
-  <xacro:include filename="$(find linorobot2_description)/urdf/sensors/depth_sensor.urdf.xacro" />
-  <xacro:include filename="$(find linorobot2_description)/urdf/controllers/diff_drive.urdf.xacro" />
+  <xacro:include filename="$(find elsabot_jeep)/urdf/mech/base.urdf.xacro" />
+  <xacro:include filename="$(find elsabot_jeep)/urdf/mech/wheel.urdf.xacro" />
+  <xacro:include filename="$(find elsabot_jeep)/urdf/mech/caster_wheel.urdf.xacro" />
+  <xacro:include filename="$(find elsabot_jeep)/urdf/sensors/imu.urdf.xacro" />
+  <xacro:include filename="$(find elsabot_jeep)/urdf/sensors/generic_laser.urdf.xacro" />
+  <xacro:include filename="$(find elsabot_jeep)/urdf/sensors/depth_sensor.urdf.xacro" />
+  <xacro:include filename="$(find elsabot_jeep)/urdf/controllers/diff_drive.urdf.xacro" />
   <xacro:property name="laser_pose">
     <origin xyz="0.0 0 0.325" rpy="-3.1416 0 0"/>

File: urdf/sensors/generic_laser.urdf.xacro (robot description, xacro)
@@ -1,5 +1,5 @@
 <?xml version="1.0"?>
 <robot xmlns:xacro="http://ros.org/wiki/xacro">
-  <xacro:include filename="$(find linorobot2_description)/urdf/sensors/laser.urdf.xacro" />
+  <xacro:include filename="$(find elsabot_jeep)/urdf/sensors/laser.urdf.xacro" />
   <xacro:macro name="generic_laser" params="*origin">
     <xacro:laser

File: urdf/sensors/imu.urdf.xacro (robot description, xacro)
@@ -5,5 +5,5 @@
       <parent link="base_link"/>
       <child link="imu_link"/>
-      <origin xyz="0 0.025 0.028" rpy="0 0 0"/>
+      <origin xyz="-0.331 0.055 0.066" rpy="0 0 0"/>
     </joint>
     <gazebo reference="imu_link">

File: urdf/sensors/oakd_on_ptbase.urdf.xacro (robot description, xacro)
@@ -42,5 +42,5 @@
     </link>
     <joint name="cam_pan_joint" type="revolute">
-      <origin xyz="-0.030 0.0 0.535" rpy="0 0 0" />
+      <origin xyz="-0.493 0.0 0.833" rpy="0 0 0" />
       <axis xyz="0 0 1"/>
       <limit upper="1.57" lower="-1.57" effort="10" velocity="10"/>
@@ -79,5 +79,5 @@
         <geometry>
           <!-- box size="${length} ${width} ${height}"/ -->
-          <mesh filename="package://linorobot2_description/meshes/oakd.stl" scale="1.0 1.0 1.0"/> -->
+          <mesh filename="package://elsabot_jeep/meshes/oakd.stl" scale="1.0 1.0 1.0"/> -->
         </geometry>
         <material name="black">
