Commit message: Add support for ultrasonic distance sensors on the back.

File: urdf/jeep_properties.urdf.xacro (robot description, xacro)
@@ -18,3 +18,9 @@
     <origin xyz="-0.065 0 0.255" rpy="0 0 0"/>
   </xacro:property>
+  <xacro:property name="range_back_left_pose">
+    <origin xyz="-0.543 0.205 0.298" rpy="0 0 -3.14"/>
+  </xacro:property>
+  <xacro:property name="range_back_right_pose">
+    <origin xyz="-0.543 -0.205 0.298" rpy="0 0 -3.14"/>
+  </xacro:property>
 </robot>

File: urdf/robots/jeep.urdf.xacro (robot description, xacro)
@@ -8,4 +8,5 @@
   <!--xacro:include filename="$(find elsabot_jeep)/urdf/sensors/depth_sensor.urdf.xacro" /-->
   <xacro:include filename="$(find elsabot_jeep)/urdf/sensors/oakd_on_ptbase.urdf.xacro" />
+  <xacro:include filename="$(find elsabot_jeep)/urdf/sensors/hcsr04.urdf.xacro" />
   <!--xacro:include filename="$(find elsabot_jeep)/urdf/controllers/skid_steer.urdf.xacro" /-->
   <xacro:base
@@ -60,8 +61,9 @@
     <xacro:insert_block name="depth_sensor_pose" />
   </xacro:depth_sensor>
-  <!--xacro:diff_drive_controller
-    wheel_separation="${wheel_pos_y * 2}"
-    wheel_radius="${wheel_radius}"
-    wheel_torque="${wheel_torque}"
-  /-->
-</robot>
+  <xacro:hcsr04_sensor frame_id="hcsr04_back_left">
+    <xacro:insert_block name="range_back_left_pose" />
+  </xacro:hcsr04_sensor>
+  <xacro:hcsr04_sensor frame_id="hcsr04_back_right">
+    <xacro:insert_block name="range_back_right_pose" />
+  </xacro:hcsr04_sensor>
+  </robot>

Commit message: WIP support for OakD as depth sensor for nav

File: urdf/jeep_properties.urdf.xacro (robot description, xacro)
@@ -24,3 +24,14 @@
     <origin xyz="-0.543 -0.205 0.298" rpy="0 0 -3.14"/>
   </xacro:property>
+  <!-- OakD as depth sensor -->
+  <xacro:property name="depth_camera_name" value="oak" />
+  <xacro:property name="depth_camera_model" value="OAK-D" />
+  <xacro:property name="depth_base_frame" value="front_oakd_base_link" />
+  <xacro:property name="depth_parent_frame" value="base_link" />
+  <xacro:property name="depth_cam_pos_x" value="0.254" />
+  <xacro:property name="depth_cam_pos_y" value="0.0" />
+  <xacro:property name="depth_cam_pos_z" value="0.620" />
+  <xacro:property name="depth_cam_roll" value="0.0" />
+  <xacro:property name="depth_cam_pitch" value="0.42" />
+  <xacro:property name="depth_cam_yaw" value="0.0" />
 </robot>

File: urdf/robots/jeep.urdf.xacro (robot description, xacro)
@@ -6,4 +6,5 @@
   <xacro:include filename="$(find elsabot_jeep)/urdf/sensors/imu.urdf.xacro" />
   <xacro:include filename="$(find elsabot_jeep)/urdf/sensors/generic_laser.urdf.xacro" />
+  <xacro:include filename="$(find elsabot_jeep)/urdf/sensors/depthai_macro.urdf.xacro" />
   <!--xacro:include filename="$(find elsabot_jeep)/urdf/sensors/depth_sensor.urdf.xacro" /-->
   <xacro:include filename="$(find elsabot_jeep)/urdf/sensors/oakd_on_ptbase.urdf.xacro" />
@@ -67,3 +68,15 @@
     <xacro:insert_block name="range_back_right_pose" />
   </xacro:hcsr04_sensor>
+  <xacro:depthai_camera
+   camera_name = "${depth_camera_name}"
+   parent = "${depth_parent_frame}"
+   camera_model = "${depth_camera_model}"
+   base_frame = "${depth_base_frame}"
+   cam_pos_x = "${depth_cam_pos_x}"
+   cam_pos_y = "${depth_cam_pos_y}"
+   cam_pos_z = "${depth_cam_pos_z}"
+   cam_roll = "${depth_cam_roll}"
+   cam_pitch = "${depth_cam_pitch}"
+   cam_yaw = "${depth_cam_yaw}"
+  />
   </robot>

Commit message: Setup Gazeobo support
Current use case is for testing Elsabot Jeep driving autonomously
in a loop.  See Readme.

File: urdf/jeep_properties.urdf.xacro (robot description, xacro)
@@ -4,5 +4,6 @@
   <xacro:property name="base_width" value="0.653" />
   <xacro:property name="base_height" value="0.450" />
-  <xacro:property name="base_mass" value="10" />
+  <xacro:property name="base_mass" value="50.0" />
+  <xacro:property name="wheel_base" value="0.708" />
   <xacro:property name="wheel_radius" value="0.140" />
   <xacro:property name="wheel_width" value="0.170" />
@@ -10,6 +11,10 @@
   <xacro:property name="wheel_pos_y" value="0.3265" />
   <xacro:property name="wheel_pos_z" value="0.0" />
-  <xacro:property name="wheel_mass" value=".6" />
+  <xacro:property name="wheel_mass" value="0.2" />
   <xacro:property name="wheel_torque" value="12" />
+  <xacro:property name="wheel_max_steer" value="0.925" />
+  <xacro:property name="wheel_mass_steering" value=".1" />
+  <xacro:property name="kingpin_width" value="0.490" />
+  <xacro:property name="wheel_center_to_kingpin" value="0.082" />
   <xacro:property name="laser_pose">
     <origin xyz="0.354 0 0.440" rpy="0 0 3.14"/>

File: urdf/mech/base.urdf.xacro (robot description, xacro)
@@ -14,10 +14,10 @@
         </material>
       </visual>
-      <collision>
+      <!--collision>
         <origin xyz="0 0 0" rpy="0 0 0"/>
         <geometry>
           <box size="${length} ${width} ${height}"/>
         </geometry>
-      </collision>
+      </collision-->
       <inertial>
         <origin xyz="0 0 0" rpy="0 0 0"/>

File: urdf/mech/wheel.urdf.xacro (robot description, xacro)
@@ -1,6 +1,15 @@
 <?xml version="1.0"?>
 <robot xmlns:xacro="http://ros.org/wiki/xacro">
-  <xacro:macro name="wheel" params="side radius width pos_x pos_y pos_z mass">
+  <xacro:macro name="wheel" params="side radius width pos_x pos_y pos_z mass parent_link">
     <link name="${side}_wheel_link">
+      <visual>
+        <origin xyz="0 0 0" rpy="${pi/2} 0 0"/>
+        <geometry>
+          <cylinder radius="${radius}" length="${width}"/>
+        </geometry>
+        <material name="blue">
+            <color rgba="0.1764 0.4588 0.8509 1.0"/>
+        </material>
+      </visual>
       <collision>
         <origin xyz="0 0 0" rpy="${pi/2} 0 0"/>
@@ -8,4 +17,12 @@
           <cylinder radius="${radius}" length="${width}"/>
         </geometry>
+        <surface>
+          <friction>
+            <ode>
+              <mu>0.5</mu>
+              <mu2>1.0</mu2>
+            </ode>
+          </friction>
+        </surface>
       </collision>
       <inertial>
@@ -29,8 +46,10 @@
     <joint name="${side}_wheel_joint" type="continuous">
       <axis xyz="0 1 0" />
-      <parent link="base_link"/>
+      <parent link="${parent_link}"/>
       <child link="${side}_wheel_link"/>
       <origin xyz="${pos_x} ${pos_y} ${pos_z}" rpy="0 0 0"/>
     </joint>
+    <gazebo reference="${side}_wheel_joint">
+    </gazebo>
   </xacro:macro>
 </robot>

File: urdf/robots/jeep.urdf.xacro (robot description, xacro)
@@ -4,11 +4,12 @@
   <xacro:include filename="$(find elsabot_jeep)/urdf/mech/base.urdf.xacro" />
   <xacro:include filename="$(find elsabot_jeep)/urdf/mech/wheel.urdf.xacro" />
+  <xacro:include filename="$(find elsabot_jeep)/urdf/mech/wheel_steering.urdf.xacro" />
   <xacro:include filename="$(find elsabot_jeep)/urdf/sensors/imu.urdf.xacro" />
   <xacro:include filename="$(find elsabot_jeep)/urdf/sensors/generic_laser.urdf.xacro" />
   <xacro:include filename="$(find elsabot_jeep)/urdf/sensors/depthai_macro.urdf.xacro" />
-  <!--xacro:include filename="$(find elsabot_jeep)/urdf/sensors/depth_sensor.urdf.xacro" /-->
   <xacro:include filename="$(find elsabot_jeep)/urdf/sensors/oakd_on_ptbase.urdf.xacro" />
   <xacro:include filename="$(find elsabot_jeep)/urdf/sensors/hcsr04.urdf.xacro" />
-  <!--xacro:include filename="$(find elsabot_jeep)/urdf/controllers/skid_steer.urdf.xacro" /-->
+  <xacro:include filename="$(find elsabot_jeep)/urdf/controllers/ackermann_drive.urdf.xacro" />
+  <!--xacro:include filename="$(find elsabot_jeep)/urdf/sensors/depth_sensor.urdf.xacro" /-->
   <xacro:base
     length="${base_length}"
@@ -18,24 +19,27 @@
     wheel_radius="${wheel_radius}"
     wheel_pos_z="${wheel_pos_z}"
-/>
+  />
   <xacro:wheel
+    parent_link="front_left_wheel_steering_link"
     side="front_left"
     radius="${wheel_radius}"
     width="${wheel_width}"
-    pos_x="${wheel_pos_x}"
-    pos_y="${wheel_pos_y}"
-    pos_z="${wheel_pos_z}"
+    pos_x="0"
+    pos_y="${wheel_center_to_kingpin}"
+    pos_z="0"
     mass="${wheel_mass}"
   />
   <xacro:wheel
+    parent_link="front_right_wheel_steering_link"
     side="front_right"
     radius="${wheel_radius}"
     width="${wheel_width}"
-    pos_x="${wheel_pos_x}"
-    pos_y="${-wheel_pos_y}"
-    pos_z="${wheel_pos_z}"
+    pos_x="0"
+    pos_y="${-wheel_center_to_kingpin}"
+    pos_z="0"
     mass="${wheel_mass}"
   />
   <xacro:wheel
+    parent_link="base_link"
     side="rear_left"
     radius="${wheel_radius}"
@@ -47,4 +51,5 @@
   />
   <xacro:wheel
+    parent_link="base_link"
     side="rear_right"
     radius="${wheel_radius}"
@@ -54,4 +59,22 @@
     pos_z="${wheel_pos_z}"
     mass="${wheel_mass}"
+  />
+  <xacro:wheel_steering
+    parent_link="base_link"
+    side="front_left"
+    pos_x="${wheel_pos_x}"
+    pos_y="${kingpin_width/2}"
+    pos_z="${wheel_pos_z}"
+    mass="${wheel_mass_steering}"
+    max_steer="${wheel_max_steer}"
+  />
+  <xacro:wheel_steering
+    parent_link="base_link"
+    side="front_right"
+    pos_x="${wheel_pos_x}"
+    pos_y="${-kingpin_width/2}"
+    pos_z="${wheel_pos_z}"
+    mass="${wheel_mass_steering}"
+    max_steer="${wheel_max_steer}"
   />
   <xacro:imu/>
@@ -80,3 +103,18 @@
    cam_yaw = "${depth_cam_yaw}"
   />
+  <gazebo>
+    <plugin filename="ignition-gazebo-joint-state-publisher-system" name="ignition::gazebo::systems::JointStatePublisher"/>
+    <plugin filename="ignition-gazebo-sensors-system" name="ignition::gazebo::systems::Sensors">
+      <render_engine>ogre2</render_engine>
+    </plugin>
+    <plugin filename="ignition-gazebo-imu-system" name="ignition::gazebo::systems::Imu">
+    </plugin>
+  </gazebo>
+  <xacro:ackermann_drive_controller
+    wheel_base = "${wheel_base}"
+    wheel_max_steer = "${wheel_max_steer}"
+    wheel_separation = "${2*wheel_pos_y}"
+    kingpin_width = "${kingpin_width}"
+    wheel_radius = "${wheel_radius}"
+  />
   </robot>

File: urdf/sensors/imu.urdf.xacro (robot description, xacro)
@@ -1,5 +1,13 @@
 <robot xmlns:xacro="http://ros.org/wiki/xacro">
   <xacro:macro name="imu">
-    <link name="imu_link"/>
+    <link name="imu_link">
+      <inertial>
+        <origin xyz="0 0 0" rpy="0 0 0"/>
+        <mass value="0.1"/>
+        <inertia ixx="0.1" ixy="0" ixz="0"
+                 iyy="0.1" iyz="0"
+                 izz="0.1" />
+      </inertial>
+    </link>
     <joint name="imu_to_base_link" type="fixed">
       <parent link="base_link"/>
@@ -9,23 +17,15 @@
     <gazebo reference="imu_link">
       <gravity>true</gravity>
-      <sensor name="imu_sensor" type="imu">
-      <always_on>true</always_on>
+      <sensor name="imu_link" type="imu">
+        <topic>imu/data</topic>
+        <frameName>imu_link</frameName>
+        <ignition_frame_id>imu_link</ignition_frame_id>
+        <always_on>1</always_on>
       <update_rate>20</update_rate>
       <visualize>true</visualize>
-      <topic>__default_topic__</topic>
-      <plugin filename="libgazebo_ros_imu_sensor.so" name="imu_plugin">
-          <ros>
-            <remapping>~/out:=imu/data</remapping>
-          </ros>
-          <topicName>imu/data</topicName>
-          <bodyName>imu_link</bodyName>
-          <updateRateHZ>10.0</updateRateHZ>
-          <gaussianNoise>0.0</gaussianNoise>
+        <gaussianNoise>0</gaussianNoise>
           <xyzOffset>0 0 0</xyzOffset>
           <rpyOffset>0 0 0</rpyOffset>
-          <frameName>imu_link</frameName>
           <initialOrientationAsReference>false</initialOrientationAsReference>
-      </plugin>
-      <pose>0 0 0 0 0 0</pose>
       </sensor>
     </gazebo>

File: urdf/sensors/laser.urdf.xacro (robot description, xacro)
@@ -42,10 +42,9 @@
     </joint>
     <gazebo reference="${frame_id}">
-      <sensor type="ray" name="${frame_id}_head_hokuyo_sensor">
-        <always_on>true</always_on>
-        <update_rate>${update_rate}</update_rate>
-        <pose>0 0 0 0 0 0</pose>
-        <visualize>false</visualize>
-        <ray>
+      <sensor name="${frame_id}" type='gpu_lidar'>
+        <topic>${topic_name}</topic>
+        <ignition_frame_id>${frame_id}</ignition_frame_id>
+        <update_rate>10</update_rate>
+        <lidar>
           <scan>
             <horizontal>
@@ -55,4 +54,10 @@
               <max_angle>${max_angle}</max_angle>
             </horizontal>
+            <vertical>
+              <samples>1</samples>
+              <resolution>0.01</resolution>
+              <min_angle>0.0</min_angle>
+              <max_angle>0.0</max_angle>
+            </vertical>
           </scan>
           <range>
@@ -61,16 +66,7 @@
             <resolution>0.01</resolution>
           </range>
-        </ray>
-        <plugin name="${frame_id}_gazebo_ros_head_hokuyo_controller" filename="libgazebo_ros_ray_sensor.so">
-          <ros>
-            <remapping>~/out:=${topic_name}</remapping>
-          </ros>
-          <output_type>sensor_msgs/LaserScan</output_type>
-          <alwaysOn>true</alwaysOn>
-          <updateRate>${update_rate}</updateRate>
-          <topicName>${topic_name}</topicName>
-          <frame_name>${frame_id}</frame_name>
-          <output_type>sensor_msgs/LaserScan</output_type>
-        </plugin>
+        </lidar>
+        <alwaysOn>1</alwaysOn>
+        <visualize>true</visualize>
       </sensor>
     </gazebo>
