Commit message: Support Accel pedal for enabling movement during nav, some misc cleanup

File: urdf/controllers/ackermann_drive.urdf.xacro (robot description, xacro)
@@ -21,5 +21,5 @@
         <odom_topic>odom</odom_topic>
         <odom_publish_frequency>20</odom_publish_frequency>
-        <topic>cmd_vel</topic>
+        <topic>cmd_vel_filtered</topic>
         <frame_id>odom</frame_id>
         <child_frame_id>base_footprint</child_frame_id>

File: urdf/mech/base.urdf.xacro (robot description, xacro)
@@ -8,5 +8,5 @@
         <geometry>
           <!-- box size="${length} ${width} ${height}"/ -->
-          <mesh filename="package://elsabot_jeep/meshes/jeep_simple.stl" scale="1.0 1.0 1.0"/> -->
+          <mesh filename="package://elsabot_jeep/meshes/jeep_simple.stl" scale="1.0 1.0 1.0"/>
         </geometry>
         <material name="gray">

File: urdf/sensors/oakd_on_ptbase.urdf.xacro (robot description, xacro)
@@ -79,5 +79,5 @@
         <geometry>
           <!-- box size="${length} ${width} ${height}"/ -->
-          <mesh filename="package://elsabot_jeep/meshes/oakd.stl" scale="1.0 1.0 1.0"/> -->
+          <mesh filename="package://elsabot_jeep/meshes/oakd.stl" scale="1.0 1.0 1.0"/>
         </geometry>
         <material name="black">

Commit message: Jazzy related changes

File: urdf/controllers/ackermann_drive.urdf.xacro (robot description, xacro)
@@ -2,5 +2,5 @@
   <xacro:macro name="ackermann_drive_controller" params="wheel_separation kingpin_width wheel_base wheel_radius wheel_max_steer">
     <gazebo>
-      <plugin name="ignition::gazebo::systems::AckermannSteering" filename="ignition-gazebo-ackermann-steering-system">
+      <plugin name="gz::sim::systems::AckermannSteering" filename="gz-sim-ackermann-steering-system">
         <left_joint>rear_left_wheel_joint</left_joint>
         <right_joint>rear_right_wheel_joint</right_joint>
@@ -16,7 +16,8 @@
         <!--max_wheel_acceleration>1.0</max_wheel_acceleration-->
         <min_velocity>-1.0</min_velocity>
-        <max_velocity>2.0</max_velocity>
+        <max_velocity>3.0</max_velocity>
         <min_acceleration>-1.0</min_acceleration>
         <max_acceleration>2.0</max_acceleration>
+        <steer_p_gain>10.0</steer_p_gain>
         <odom_topic>odom</odom_topic>
         <odom_publish_frequency>20</odom_publish_frequency>

File: urdf/controllers/diff_drive.urdf.xacro (robot description, xacro)
@@ -2,5 +2,5 @@
   <xacro:macro name="diff_drive_controller" params="wheel_separation wheel_radius wheel_torque">
     <gazebo>
-      <plugin name="differential_drive_controller" filename="libgazebo_ros_diff_drive.so">
+      <plugin name="differential_drive_controller" filename="gz-sim-ros-diff-drive">
         <ros>
           <argument>odom:=odom/unfiltered</argument>

File: urdf/controllers/omni_drive.urdf.xacro (robot description, xacro)
@@ -2,5 +2,5 @@
   <xacro:macro name="omni_drive_controller">
     <gazebo>
-    <plugin name="object_controller" filename="libgazebo_ros_planar_move.so">
+    <plugin name="object_controller" filename="gz-sim-ros-planar-move">
       <ros>
         <argument>odom:=odom/unfiltered</argument>

File: urdf/controllers/skid_steer.urdf.xacro (robot description, xacro)
@@ -2,5 +2,5 @@
   <xacro:macro name="diff_drive_controller" params="wheel_separation wheel_radius wheel_torque">
     <gazebo>
-      <plugin name="differential_drive_controller" filename="libgazebo_ros_diff_drive.so">
+      <plugin name="differential_drive_controller" filename="gz-sim-ros-diff-drive">
         <ros>
           <argument>odom:=odom/unfiltered</argument>

File: urdf/jeep_properties.urdf.xacro (robot description, xacro)
@@ -13,5 +13,5 @@
   <xacro:property name="wheel_mass" value="0.2" />
   <xacro:property name="wheel_torque" value="12" />
-  <xacro:property name="wheel_max_steer" value="0.925" />
+  <xacro:property name="wheel_max_steer" value="0.435" />
   <xacro:property name="wheel_mass_steering" value=".1" />
   <xacro:property name="kingpin_width" value="0.490" />

File: urdf/robots/jeep.urdf.xacro (robot description, xacro)
@@ -104,9 +104,9 @@
   />
   <gazebo>
-    <plugin filename="ignition-gazebo-joint-state-publisher-system" name="ignition::gazebo::systems::JointStatePublisher"/>
-    <plugin filename="ignition-gazebo-sensors-system" name="ignition::gazebo::systems::Sensors">
+    <plugin filename="gz-sim-joint-state-publisher-system" name="gz::sim::systems::JointStatePublisher"/>
+    <plugin filename="gz-sim-sensors-system" name="gz::sim::systems::Sensors">
       <render_engine>ogre2</render_engine>
     </plugin>
-    <plugin filename="ignition-gazebo-imu-system" name="ignition::gazebo::systems::Imu">
+    <plugin filename="gz-sim-imu-system" name="gz::sim::systems::Imu">
     </plugin>
   </gazebo>

File: urdf/sensors/depth_sensor.urdf.xacro (robot description, xacro)
@@ -61,5 +61,5 @@
           </image>
         </camera>
-        <plugin name="camera_controller" filename="libgazebo_ros_camera.so">
+        <plugin name="camera_controller" filename="gz-sim-ros-camera">
           <ros>
             <remapping>/camera/camera_info:=/camera/color/camera_info</remapping>

File: urdf/sensors/imu.urdf.xacro (robot description, xacro)
@@ -20,5 +20,5 @@
         <topic>imu/data</topic>
         <frameName>imu_link</frameName>
-        <ignition_frame_id>imu_link</ignition_frame_id>
+        <gz_frame_id>imu_link</gz_frame_id>
         <always_on>1</always_on>
       <update_rate>20</update_rate>

File: urdf/sensors/laser.urdf.xacro (robot description, xacro)
@@ -44,5 +44,5 @@
       <sensor name="${frame_id}" type='gpu_lidar'>
         <topic>${topic_name}</topic>
-        <ignition_frame_id>${frame_id}</ignition_frame_id>
+        <gz_frame_id>${frame_id}</gz_frame_id>
         <update_rate>10</update_rate>
         <lidar>
